File: Ardui89_Uno_Board/Ardui89_Uno.kicad_pcb (KiCad board)
At the start: 2 copper layers, 68.8 x 53.5 mm, 47 parts, among them J1 Jack-DC, J101 Conn_01x19, J102 Conn_01x16, J201 USB_TYPE_B, Q101 BC856, SW101 SW_Push, U1 LD1117S50TR, U101 STC15C2K16/32-DIP28, U2 LP2985-33DBVR, U201 CH340G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

Commit message: Add files via upload
Parts:
- added D202: 1N4148W, Diode_SMD:D_1206_3216Metric_Pad1.42x1.75mm_HandSolder, F.Cu at (136.4, 97.7)
- C100, C101, C203: value 0.1µ -> 100n
- C3: value 0.1 uF -> 100n
- R1: value 510 -> 1K
- R130, R201, R202: value 510 -> 1k
- U101: value STC15C2K16/32-DIP28 -> STC15F2K16/32-DIP28
- moved G*** 24.0 mm to (144.7, 113.0)
- moved R1 8.41 mm to (144.8, 97.3), turned to 90 degrees
- moved D1 8.20 mm to (144.8, 91.7)
- moved C4 3.06 mm to (140.0, 97.7)
- moved C200 1.91 mm to (140.2, 90.8)
- moved G*** 1.14 mm to (158.0, 91.1)
- moved D200 0.51 mm to (136.4, 90.8)
- turned D_Rx201 to 90 degrees
- turned R202 to -90 degrees
Connections:
- D_Rx201 pad 1: Net-(D_Rx201-K) -> /Rx
- D_Rx201 pad 2: /Rx -> Net-(D_Rx201-A)
- D_Tx202 pad 1: Net-(D_Tx201-K) -> Net-(D_Tx202-K)
- R201 pad 1: Net-(D_Rx201-K) -> VCC
- R201 pad 2: GND -> Net-(D_Rx201-A)
- R202 pad 1: Net-(D_Tx201-K) -> Net-(D202-A)
- R202 pad 2: GND -> Net-(D_Tx202-K)
- U1 pad 4: GND -> (no net)
Routing:
- net VCC: track 207.4 -> 199.2 mm
- net Net-(D202-A): track 0.00 -> 6.55 mm
- net Net-(D_Tx202-K): track 0.00 -> 4.04 mm
- net Net-(D_Tx201-K): track 4.04 -> 0.00 mm
- net Net-(D_Rx201-K): track 4.04 -> 0.00 mm
- net Net-(D_Rx201-A): track 0.00 -> 2.44 mm
- net Net-(D200-A): track 4.83 -> 4.27 mm
- net Net-(D1-A): track 3.07 -> 2.55 mm
- net GND: vias 8 -> 9
Other:
- board text added: "L"
- board text added: "ON"
