File: Ardui89_Uno_Board/Ardui89_Uno.kicad_sch (KiCad schematic)
At the start: 45 parts, among them J1 Jack-DC, J101 Conn_01x19, J102 Conn_01x16, J201 USB_TYPE_B, Q101 BC856, SW101 SW_Push, U1 LD1117S50TR, U101 STC15F2K16/32-DIP28, U2 LP2985-33DBVR, U201 CH340G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

Commit message: Add files via upload
Parts:
- added D202: 1N4148W, Diode_SMD:D_1206_3216Metric_Pad1.42x1.75mm_HandSolder, symbol Diode:1N4148W
- C100, C101, C203: value 0.1µ -> 100n
- C3: value 0.1 uF -> 100n
- R1: value 510 -> 1K
- R130, R201, R202: value 510 -> 1k
Connections:
- net GND: now also D202.1 (K); no longer R201.2, R202.2, U1.4 (GND)
- net Rx: now also D_Rx201.1 (K); no longer D_Rx201.2 (A)
- net VCC: now also R201.1
- net at D_Tx202.1 (K): now also R202.2; no longer R202.1
- new net: D_Rx201.2 (A), R201.2
- new net: D202.2 (A), R202.1
Other:
- moved on the sheet: D_Rx201, D_Tx202, R201, R202
